Commit message: ultrasónico añadido y funciona

File: comm/ros2/mounted/ws/src/sim/robot.urdf (robot description, URDF)
Before this commit: robot lego_ev3, 6 links, 5 joints
Joints:
- joint base_ultrasonic_joint: origin xyz=-0.3 0 0.15 rpy=0 0 0 -> xyz=-0.3 0 0.15 rpy=0 0 3.14

Commit message: girosensor añadido

File: comm/ros2/mounted/ws/src/sim/robot.urdf (robot description, URDF)
Before this commit: robot lego_ev3, 6 links, 5 joints
Links:
- added link base_gyro
Joints:
- added joint base_gyro_joint: type continuous, parent base_gyro, child base_link, origin xyz=0 0 0 rpy=0 0 0, axis 0 0 1
- joint base_joint: child base_link -> base_gyro

Commit message: urdf: sensores de color ev3

File: comm/ros2/mounted/ws/src/sim/robot.urdf (robot description, URDF)
Before this commit: robot lego_ev3, 7 links, 6 joints
Links:
- added link left_color_light_sensor; visual box size=0.04 0.04 0.08
- added link right_color_light_sensor; visual box size=0.04 0.04 0.08
Joints:
- added joint base_left_color_light_sensor_joint: type fixed, parent base_link, child left_color_light_sensor, origin xyz=-0.28 0.18 0.01 rpy=0 0 3.14
- added joint base_right_color_light_sensor_joint: type fixed, parent base_link, child right_color_light_sensor, origin xyz=-0.28 -0.18 0.01 rpy=0 0 3.14

Commit message: sensores de color en ROS2 y su halo en RVIZ, hecho

File: comm/ros2/mounted/ws/src/sim/robot.urdf (robot description, URDF)
Before this commit: robot lego_ev3, 9 links, 8 joints
Joints:
- joint base_left_color_light_sensor_joint: origin xyz=-0.28 0.18 0.01 rpy=0 0 3.14 -> xyz=-0.28 -0.18 0.01 rpy=0 0 3.14
- joint base_right_color_light_sensor_joint: origin xyz=-0.28 -0.18 0.01 rpy=0 0 3.14 -> xyz=-0.28 0.18 0.01 rpy=0 0 3.14
